File: pcb/ice6502.kicad_pcb (KiCad board)
At the start: 2 copper layers, 100 x 50 mm, 54 parts, among them J1 Programming Header, J2 RDY, J3 RESB, J4 VIN, J5 GND, J6 3v3, J7 1v2, J8 GND, U0 iCE40-HX4K-TQ144, U1 AT25SF041-SSHD-B, U1_1 W65C816S_PLCC, U2 VXO7803-1000, U3 IS61WV5128EDBLL-10TLI, X1 ASE-xxxMHz

Commit message: Continue on pcb
Parts:
- R6, R7: moved to F.Cu
- moved C6 12.8 mm to (113.0, 87.0), turned to 90 degrees
- moved X1 11.8 mm to (113.0, 87.0), turned to 90 degrees
- moved C5 10.5 mm to (121.0, 81.0)
- moved R6 6.82 mm to (121.0, 87.0), turned to 90 degrees
- moved R7 4.94 mm to (123.0, 87.0), turned to 90 degrees
- moved U1 4.47 mm to (121.0, 81.0), turned to 0 degrees
- moved R5 3.86 mm to (120.0, 77.2)
- moved R2 3.01 mm to (116.8, 87.0), turned to 90 degrees
- moved R1 2.80 mm to (118.8, 87.0), turned to 90 degrees
- moved J1 1.12 mm to (138.5, 93.5)
Connections:
- net N$2 renamed CRESET_B
- net N$3 renamed CDONE
- R6 pad 2: N$9 (its old number) -> ~WP
- R7 pad 2: N$10 (its old number) -> ~HOLD
- U1 pad 3: N$9 (its old number) -> ~WP
- U1 pad 7: N$10 (its old number) -> ~HOLD
Routing:
- net CDONE: track 0.00 -> 9.21 mm
- net ~HOLD: track 0.00 -> 7.46 mm
- net N$7: track 0.00 -> 6.35 mm
- net ~WP: track 0.00 -> 5.41 mm
- net PLLGND: track 6.90 -> 2.12 mm, vias 1 -> 0
- net 3v3: track 92.5 -> 95.9 mm, vias 4 -> 6
- net GND: track 24.1 -> 26.6 mm, vias 11 -> 13
- net MOSI: track 13.5 -> 14.6 mm
- net SCK: track 13.5 -> 12.7 mm
- net CRESET_B: track 9.61 -> 10.2 mm

Commit message: wip2
Parts:
- J3: value RESB -> ~RES
Connections:
- net CRESET_B renamed ~CRESET
- net RESB renamed ~RES
- U0 pad 31: (no net) -> ~ABORT
- U0 pad 32: (no net) -> VDA
- U0 pad 33: (no net) -> VPA
- U0 pad 34: (no net) -> ~VP
- U1_1 pad 2: (no net) -> ~VP
- U1_1 pad 4: (no net) -> ~ABORT
- U1_1 pad 43: (no net) -> VDA
- U1_1 pad 8: (no net) -> VPA
Routing:
- net 3v3: track 95.9 -> 98.6 mm

Commit message: Last commit for this revision
Parts:
- added U4: STP16CP05, TSSOP-24_4.4x7.8mm_Pitch0.65mm, B.Cu at (107.5, 60.0)
- U3: moved to B.Cu
- moved U3 10.3 mm to (120.0, 62.5), turned to 270 degrees
- moved C5 7.91 mm to (123.5, 88.5)
- moved R1 7.91 mm to (121.2, 94.5)
- moved R2 7.91 mm to (119.2, 94.5)
- moved R5 7.91 mm to (122.5, 84.8)
- moved R6 7.91 mm to (123.5, 94.5)
- moved R7 7.91 mm to (125.5, 94.5)
- moved U1 7.91 mm to (123.5, 88.5)
Connections:
- U0 pad 128: (no net) -> VDA
- U0 pad 31: ~ABORT -> (no net)
- U0 pad 32: VDA -> ~ABORT
Routing:
- net addr_b10: track 33.1 -> 0.00 mm
- net addr_b9: track 32.5 -> 0.00 mm
- net addr_b11: track 32.4 -> 0.00 mm
- net addr_b12: track 31.9 -> 0.00 mm
- net addr_b13: track 31.5 -> 0.00 mm
- net addr_b14: track 31.3 -> 0.00 mm
- net addr_b8: track 31.2 -> 0.00 mm
- net addr_b16: track 30.6 -> 0.00 mm
- net addr_b17: track 30.6 -> 0.00 mm
- net addr_b15: track 30.4 -> 0.00 mm
- net addr_b7: track 30.1 -> 0.00 mm
- net addr_b6: track 28.9 -> 0.00 mm
- net addr_b5: track 27.8 -> 0.00 mm
- net addr_b18: track 20.6 -> 0.00 mm
- net addr_b4: track 20.3 -> 0.00 mm
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